File: flex/quacken.kicad_pcb (KiCad board)
At the start: 2 copper layers, 258.8 x 111.5 mm, 111 parts, among them J1 CIRQUE_Left, J2 CIRQUE_Right, J3 USB_C_Receptacle_USB2.0_16P, U1 W25Q128JVS, U2 RP2040, U3 PCAL6524HEAZ, U4 XC6206PxxxMR, U5 SRV05-4, Y1 12MHz 18pF

Commit message: flex 25.11 (#11)
Parts:
- removed G***: LOGO, LOGO
- removed MS1, MS10, MS11, MS12, MS2 (x2), MS3, MS4, MS5, MS6, MS7, MS8, MS9: ~, keyboard:MedianPosition
- removed R11: 22k, Resistor_SMD:R_0402_1005Metric
- removed REF** (x2): MountingHole_2.2mm_M2, MountingHole:MountingHole_2.2mm_M2
- removed the SW2 at (-117.0, 89.2) (x2)
- removed the SW2 at (-86.8, 89.2)
- removed the SW2 at (60.5, 96.6)
- removed the SW2 at (-147.3, 89.0)
- removed the SW3 at (-86.8, 106.2)
- removed the SW3 at (-117.0, 106.2)
- removed the SW3 at (60.5, 113.6)
- removed the SW3 at (-147.3, 106.0)
- added ?: , keyboard:Outline, F.Cu at (219.8, 95.6)
- added SW2: ~, keyboard:Choc_Switch_Median, F.Cu at (100.1, 82.8)
- added SW3: ~, keyboard:Choc_Switch, F.Cu at (100.1, 99.8)
- added U6: SRV05-4, Package_TO_SOT_SMD:SOT-23-6, F.Cu at (297.3, 112.0)
- R10, R7, R8, R9: value 22k -> 4.7k
- SW1, SW16, SW17, SW23, SW24, SW25, SW26, SW38, SW39, SW5, SW6: footprint keyboard:PG1350 -> keyboard:Choc_Switch_Median
- SW10, SW11, SW12, SW13, SW14, SW15, SW18, SW19, SW20, SW21, SW22, SW27, SW28, SW29, SW30, SW31, SW32, SW33, SW34, SW35, SW36, SW37, SW4, SW40, SW41, SW42, SW7, SW8, SW9: footprint keyboard:PG1350 -> keyboard:Choc_Switch
- moved SMDSW1 85.3 mm to (147.5, 118.9), turned to -10 degrees
- moved R13 72.8 mm to (127.8, 116.5), turned to 80 degrees
- moved R12 69.8 mm to (128.2, 114.4), turned to -100 degrees
- moved U5 68.5 mm to (130.9, 115.7), turned to -10 degrees
- moved TRRS1 58.8 mm to (217.2, 127.7), turned to -90 degrees
- moved J3 53.4 mm to (126.6, 44.0)
- moved C6 49.9 mm to (152.3, 109.0), turned to 80 degrees
- moved TRRS2 46.9 mm to (222.3, 123.0), turned to 90 degrees
- moved U1 45.5 mm to (154.7, 113.5), turned to 80 degrees
- moved C10 45.5 mm to (151.6, 110.9), turned to -100 degrees
- moved C3 44.1 mm to (142.8, 118.2), turned to -100 degrees
- moved C12 44.1 mm to (141.8, 118.0), turned to 80 degrees
- moved R3 44.1 mm to (140.8, 117.8), turned to -100 degrees
- moved R4 44.1 mm to (139.8, 117.6), turned to -100 degrees
- moved C9 44.0 mm to (143.1, 116.3), turned to 80 degrees
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Connections:
- U3 pad 26: Net-(U3-ADDR) -> +3V3
- U5 pad 5: +5V -> +3V3
Routing:
- net Net-(R5-Pad2): track 96.2 -> 2.07 mm, vias 2 -> 0
- net Net-(J3-CC1): track 8.55 -> 68.0 mm
- net Net-(J3-CC2): track 12.1 -> 70.2 mm
- net +3V3: track 288.9 -> 259.7 mm, vias 11 -> 16
- net +5V: track 97.3 -> 71.4 mm
- net /I2C0_SCL: track 218.8 -> 198.8 mm, vias 3 -> 8
- net /I2C0_SDA: track 218.8 -> 201.3 mm, vias 4 -> 9
- net Net-(U2-GPIO3): track 52.4 -> 36.5 mm
- net /rotary_left_a: track 92.5 -> 77.6 mm
- net Net-(U3-P0_2): track 61.6 -> 76.2 mm
- net Net-(U2-GPIO4): track 74.4 -> 59.9 mm
- net Net-(U2-GPIO21): track 84.1 -> 98.6 mm
- net Net-(U2-GPIO16): track 51.0 -> 65.0 mm
- net Net-(U3-P0_3): track 76.2 -> 89.9 mm
- net Net-(U2-GPIO2): track 29.5 -> 15.8 mm
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Other:
- board size 258.8 x 111.5 mm -> 262 x 112.6 mm
- board text removed: ">o_/"
- board text removed: "Quacken Split v0"

Commit message: flex 25.12
Parts:
- removed the ? at (219.8, 95.6)
- added ?: , clipboard:66bca75f-7d73-44ee-ad14-b083a89b6a44, F.Cu at (330.5, 106.9)
- added ?: , clipboard:7a87b8cf-9aff-4f5e-af7c-10d41d278be2, F.Cu at (219.5, 125.1)
- added ?: , clipboard:66bca75f-7d73-44ee-ad14-b083a89b6a44, F.Cu at (108.1, 106.9)
- added ?: , clipboard:6155f7aa-606b-4f9a-9a74-7124771ae546, F.Cu at (220.4, 58.2)
- added C19: 100n, Capacitor_SMD:C_0402_1005Metric, F.Cu at (153.4, 115.8)
- added C20: 100n, Capacitor_SMD:C_0402_1005Metric, F.Cu at (153.8, 107.3)
- added H1: TentingPuckLeft, keyboard:TentingPuck, F.Cu at (167.7, 74.7)
- added H10: MountingHole, MountingHole:MountingHole_2.2mm_M2_DIN965_Pad_TopOnly, B.Cu at (226.8, 62.1)
- added H11: MountingHole, MountingHole:MountingHole_2.2mm_M2_DIN965_Pad_TopOnly, B.Cu at (226.8, 131.1)
- added H12: MountingHole, MountingHole:MountingHole_2.2mm_M2_DIN965_Pad_TopOnly, B.Cu at (321.8, 110.6)
- added H2: TentingPuckRight, keyboard:TentingPuck, F.Cu at (270.4, 74.6)
- added H3: MountingHole, MountingHole:MountingHole_2.2mm_M2_DIN965_Pad_TopOnly, B.Cu at (98.4, 52.9)
- added H4: MountingHole, MountingHole:MountingHole_2.2mm_M2_DIN965_Pad_TopOnly, B.Cu at (115.8, 50.6)
- added H5: MountingHole, MountingHole:MountingHole_2.2mm_M2_DIN965_Pad_TopOnly, B.Cu at (210.8, 62.1)
- added H6: MountingHole, MountingHole:MountingHole_2.2mm_M2_DIN965_Pad_TopOnly, B.Cu at (115.8, 110.6)
- added H7: MountingHole, MountingHole:MountingHole_2.2mm_M2_DIN965_Pad_TopOnly, B.Cu at (210.8, 131.1)
- added H8: MountingHole, MountingHole:MountingHole_2.2mm_M2_DIN965_Pad_TopOnly, B.Cu at (340.2, 52.9)
- added H9: MountingHole, MountingHole:MountingHole_2.2mm_M2_DIN965_Pad_TopOnly, B.Cu at (321.8, 50.6)
- added J4: Qwiic, Connector_JST:JST_SH_SM04B-SRSS-TB_1x04-1MP_P1.00mm_Horizontal, F.Cu at (312.0, 46.2)
- added R11: 2.2k, Resistor_SMD:R_0402_1005Metric, F.Cu at (143.5, 112.6)
- added R2: 2.2k, Resistor_SMD:R_0402_1005Metric, F.Cu at (143.7, 111.5)
- added U7: LTC4311, Package_TO_SOT_SMD:SOT-363_SC-70-6_Handsoldering, F.Cu at (298.9, 110.8)
- C11: footprint Capacitor_SMD:C_0402_1005Metric -> Capacitor_SMD:C_0402_1005Metric_Pad0.74x0.62mm_HandSolder
- R7, R8: value 4.7k -> 2.2k
- U5: value SRV05-4 -> ECMF02-2AMX6; footprint Package_TO_SOT_SMD:SOT-23-6 -> Package_DFN_QFN:ST_UQFN-6L_1.5x1.7mm_P0.5mm
- moved C11 163.0 mm to (302.1, 110.8), turned to 100 degrees
- moved R5 20.3 mm to (133.4, 111.9), turned to 80 degrees
- moved R6 18.9 mm to (134.5, 112.1), turned to -100 degrees
- moved C6 17.6 mm to (135.4, 104.4), turned to 170 degrees
- moved SMDSW1 16.8 mm to (134.7, 107.9), turned to -100 degrees
- moved U1 15.8 mm to (139.6, 108.8)
- moved R1 14.7 mm to (152.4, 117.7)
- moved C1 14.6 mm to (152.1, 119.7)
- moved Y1 14.5 mm to (149.8, 118.2), turned to 80 degrees
- moved C2 14.5 mm to (153.2, 119.9), turned to -100 degrees
- moved C3 13.5 mm to (148.7, 106.0), turned to 80 degrees
- moved C14 11.2 mm to (149.8, 106.2), turned to 80 degrees
- moved C4 11.1 mm to (147.7, 116.4), turned to -100 degrees
- moved U5 10.4 mm to (141.3, 116.6), turned to 80 degrees
- moved C10 8.63 mm to (147.3, 118.4)
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Connections:
- J3 pad A6: /D+ -> /USB_D+
- J3 pad A7: /D- -> /USB_D-
- J3 pad B6: /D+ -> /USB_D+
- J3 pad B7: /D- -> /USB_D-
- R3 pad 2: /D+ -> /MCU_D+
- R4 pad 2: /D- -> /MCU_D-
- TRRS1 pad R1: /I2C0_SDA -> +3V3
- TRRS1 pad R2: +3V3 -> /I2C0_SDA
- TRRS2 pad R1: /I2C0_SDA -> +3V3
- TRRS2 pad R2: +3V3 -> /I2C0_SDA
- U5 pad 1: /D- -> /MCU_D+
- U5 pad 2: GND -> /MCU_D-
- U5 pad 3: /D+ -> GND
- U5 pad 4: /D- -> unconnected-(U5-NC-Pad4)
- U5 pad 5: +3V3 -> /USB_D-
- U5 pad 6: /D+ -> /USB_D+
- U6 pad 4: /I2C0_SCL -> /I2C0_SDA
- U6 pad 6: /I2C0_SDA -> /I2C0_SCL
Routing:
- net +3V3: track 259.7 -> 363.6 mm, vias 16 -> 22
- net /I2C0_SDA: track 201.3 -> 295.8 mm, vias 9 -> 11
- net /I2C0_SCL: track 198.8 -> 292.3 mm, vias 8 -> 11
- net /D+: track 88.0 -> 0.00 mm, vias 2 -> 0
- net /USB_D-: track 0.00 -> 85.2 mm, vias 0 -> 2
- net /D-: track 84.1 -> 0.00 mm, vias 4 -> 0
- net /USB_D+: track 0.00 -> 81.9 mm, vias 0 -> 2
- net GND: track 28.7 -> 52.7 mm, vias 72 -> 130
- net Net-(U3-P2_5): track 64.3 -> 47.0 mm
- net Net-(U3-P2_4): track 88.1 -> 71.2 mm
- net Net-(U2-GPIO16): track 65.0 -> 81.5 mm, vias 0 -> 2
- net +5V: track 71.4 -> 86.1 mm
- net Net-(U3-P2_6): track 41.2 -> 26.7 mm
- net /QSPI_SS: track 10.3 -> 24.1 mm
- net Net-(U2-GPIO13): track 56.0 -> 68.2 mm
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Other:
- board size 262 x 112.6 mm -> 262 x 109.6 mm
