File: flex/quacken.kicad_pcb (KiCad board)
At the start: 2 copper layers, 262 x 112.6 mm, 89 parts, among them J1 CIRQUE_Left, J2 CIRQUE_Right, J3 USB_C_Receptacle_USB2.0_16P, U1 W25Q128JVS, U2 RP2040, U3 PCAL6524HEAZ, U4 XC6206PxxxMR, U5 SRV05-4, U6 SRV05-4, Y1 12MHz 18pF

Commit message: flex 25.12 (#12)
Parts:
- removed the ? at (219.8, 95.6)
- added ?: , clipboard:66bca75f-7d73-44ee-ad14-b083a89b6a44, F.Cu at (330.5, 106.9)
- added ?: , clipboard:7a87b8cf-9aff-4f5e-af7c-10d41d278be2, F.Cu at (219.5, 125.1)
- added ?: , clipboard:66bca75f-7d73-44ee-ad14-b083a89b6a44, F.Cu at (108.1, 106.9)
- added ?: , clipboard:6155f7aa-606b-4f9a-9a74-7124771ae546, F.Cu at (220.4, 58.2)
- added C19: 100n, Capacitor_SMD:C_0402_1005Metric, F.Cu at (153.4, 115.8)
- added C20: 100n, Capacitor_SMD:C_0402_1005Metric, F.Cu at (153.8, 107.3)
- added H1: TentingPuckLeft, keyboard:TentingPuck, F.Cu at (167.7, 74.7)
- added H10: MountingHole, MountingHole:MountingHole_2.2mm_M2_DIN965_Pad_TopOnly, B.Cu at (226.8, 62.1)
- added H11: MountingHole, MountingHole:MountingHole_2.2mm_M2_DIN965_Pad_TopOnly, B.Cu at (226.8, 131.1)
- added H12: MountingHole, MountingHole:MountingHole_2.2mm_M2_DIN965_Pad_TopOnly, B.Cu at (321.8, 110.6)
- added H2: TentingPuckRight, keyboard:TentingPuck, F.Cu at (270.4, 74.6)
- added H3: MountingHole, MountingHole:MountingHole_2.2mm_M2_DIN965_Pad_TopOnly, B.Cu at (98.4, 52.9)
- added H4: MountingHole, MountingHole:MountingHole_2.2mm_M2_DIN965_Pad_TopOnly, B.Cu at (115.8, 50.6)
- added H5: MountingHole, MountingHole:MountingHole_2.2mm_M2_DIN965_Pad_TopOnly, B.Cu at (210.8, 62.1)
- added H6: MountingHole, MountingHole:MountingHole_2.2mm_M2_DIN965_Pad_TopOnly, B.Cu at (115.8, 110.6)
- added H7: MountingHole, MountingHole:MountingHole_2.2mm_M2_DIN965_Pad_TopOnly, B.Cu at (210.8, 131.1)
- added H8: MountingHole, MountingHole:MountingHole_2.2mm_M2_DIN965_Pad_TopOnly, B.Cu at (340.2, 52.9)
- added H9: MountingHole, MountingHole:MountingHole_2.2mm_M2_DIN965_Pad_TopOnly, B.Cu at (321.8, 50.6)
- added J4: Qwiic, Connector_JST:JST_SH_SM04B-SRSS-TB_1x04-1MP_P1.00mm_Horizontal, F.Cu at (312.0, 46.2)
- added R11: 2.2k, Resistor_SMD:R_0402_1005Metric, F.Cu at (143.5, 112.6)
- added R2: 2.2k, Resistor_SMD:R_0402_1005Metric, F.Cu at (143.7, 111.5)
- added U7: LTC4311, Package_TO_SOT_SMD:SOT-363_SC-70-6_Handsoldering, F.Cu at (298.9, 110.8)
- C11: footprint Capacitor_SMD:C_0402_1005Metric -> Capacitor_SMD:C_0402_1005Metric_Pad0.74x0.62mm_HandSolder
- R7, R8: value 4.7k -> 2.2k
- U5: value SRV05-4 -> ECMF02-2AMX6; footprint Package_TO_SOT_SMD:SOT-23-6 -> Package_DFN_QFN:ST_UQFN-6L_1.5x1.7mm_P0.5mm
- moved C11 163.0 mm to (302.1, 110.8), turned to 100 degrees
- moved R5 20.3 mm to (133.4, 111.9), turned to 80 degrees
- moved R6 18.9 mm to (134.5, 112.1), turned to -100 degrees
- moved C6 17.6 mm to (135.4, 104.4), turned to 170 degrees
- moved SMDSW1 16.8 mm to (134.7, 107.9), turned to -100 degrees
- moved U1 15.8 mm to (139.6, 108.8)
- moved R1 14.7 mm to (152.4, 117.7)
- moved C1 14.6 mm to (152.1, 119.7)
- moved Y1 14.5 mm to (149.8, 118.2), turned to 80 degrees
- moved C2 14.5 mm to (153.2, 119.9), turned to -100 degrees
- moved C3 13.5 mm to (148.7, 106.0), turned to 80 degrees
- moved C14 11.2 mm to (149.8, 106.2), turned to 80 degrees
- moved C4 11.1 mm to (147.7, 116.4), turned to -100 degrees
- moved U5 10.4 mm to (141.3, 116.6), turned to 80 degrees
- moved C10 8.63 mm to (147.3, 118.4)
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Connections:
- J3 pad A6: /D+ -> /USB_D+
- J3 pad A7: /D- -> /USB_D-
- J3 pad B6: /D+ -> /USB_D+
- J3 pad B7: /D- -> /USB_D-
- R3 pad 2: /D+ -> /MCU_D+
- R4 pad 2: /D- -> /MCU_D-
- TRRS1 pad R1: /I2C0_SDA -> +3V3
- TRRS1 pad R2: +3V3 -> /I2C0_SDA
- TRRS2 pad R1: /I2C0_SDA -> +3V3
- TRRS2 pad R2: +3V3 -> /I2C0_SDA
- U5 pad 1: /D- -> /MCU_D+
- U5 pad 2: GND -> /MCU_D-
- U5 pad 3: /D+ -> GND
- U5 pad 4: /D- -> unconnected-(U5-NC-Pad4)
- U5 pad 5: +3V3 -> /USB_D-
- U5 pad 6: /D+ -> /USB_D+
- U6 pad 4: /I2C0_SCL -> /I2C0_SDA
- U6 pad 6: /I2C0_SDA -> /I2C0_SCL
Routing:
- net +3V3: track 259.7 -> 363.6 mm, vias 16 -> 22
- net /I2C0_SDA: track 201.3 -> 295.8 mm, vias 9 -> 11
- net /I2C0_SCL: track 198.8 -> 292.3 mm, vias 8 -> 11
- net /D+: track 88.0 -> 0.00 mm, vias 2 -> 0
- net /USB_D-: track 0.00 -> 85.2 mm, vias 0 -> 2
- net /D-: track 84.1 -> 0.00 mm, vias 4 -> 0
- net /USB_D+: track 0.00 -> 81.9 mm, vias 0 -> 2
- net GND: track 28.7 -> 52.7 mm, vias 72 -> 130
- net Net-(U3-P2_5): track 64.3 -> 47.0 mm
- net Net-(U3-P2_4): track 88.1 -> 71.2 mm
- net Net-(U2-GPIO16): track 65.0 -> 81.5 mm, vias 0 -> 2
- net +5V: track 71.4 -> 86.1 mm
- net Net-(U3-P2_6): track 41.2 -> 26.7 mm
- net /QSPI_SS: track 10.3 -> 24.1 mm
- net Net-(U2-GPIO13): track 56.0 -> 68.2 mm
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Other:
- board size 262 x 112.6 mm -> 262 x 109.6 mm

Commit message: flex 26.01 (#15)
Parts:
- removed C11: 100n, Capacitor_SMD:C_0402_1005Metric_Pad0.74x0.62mm_HandSolder
- removed U7: LTC4311, Package_TO_SOT_SMD:SOT-363_SC-70-6_Handsoldering
- C1, C2: value 27p -> 15p
- SMDSW1: footprint keyboard:small_smd_switch -> Button_Switch_SMD:SW_SPST_TS-1088-xR020
- U1: value W25Q128JVS -> W25Q16JVUX; footprint Package_SO:SOIC-8_5.3x5.3mm_P1.27mm -> Package_SON:Winbond_USON-8-1EP_3x2mm_P0.5mm_EP0.2x1.6mm
- U5: value ECMF02-2AMX6 -> SRV05-4; footprint Package_DFN_QFN:ST_UQFN-6L_1.5x1.7mm_P0.5mm -> Package_TO_SOT_SMD:SOT-23-6
- Y1: value 12MHz 18pF -> 12MHz 10pF
- moved C2 20.5 mm to (141.1, 103.4), turned to 170 degrees
- moved C6 19.3 mm to (150.4, 116.5), turned to 80 degrees
- moved C1 19.0 mm to (147.5, 101.3), turned to -10 degrees
- moved Y1 17.7 mm to (144.1, 101.5), turned to 170 degrees
- moved C19 17.1 mm to (139.0, 106.5), turned to 170 degrees
- moved R1 16.8 mm to (143.1, 103.7), turned to -10 degrees
- moved C17 15.7 mm to (150.9, 112.9)
- moved R11 12.6 mm to (137.2, 101.7), turned to -100 degrees
- moved U1 11.1 mm to (148.6, 115.3), turned to -100 degrees
- moved R2 11.0 mm to (138.4, 101.9), turned to -100 degrees
- moved C12 10.9 mm to (141.8, 107.2), turned to 170 degrees
- moved C14 10.3 mm to (144.4, 115.1), turned to -100 degrees
- moved C15 9.87 mm to (137.3, 106.7), turned to 80 degrees
- moved C13 8.31 mm to (147.6, 103.1), turned to 80 degrees
- moved U4 7.21 mm to (138.7, 108.8), turned to 170 degrees
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Connections:
- R3 pad 2: /MCU_D+ -> /USB_D+
- R4 pad 2: /MCU_D- -> /USB_D-
- U5 pad 1: /MCU_D+ -> /USB_D-
- U5 pad 2: /MCU_D- -> GND
- U5 pad 3: GND -> /USB_D+
- U5 pad 4: unconnected-(U5-NC-Pad4) -> /USB_D+
- U5 pad 5: /USB_D- -> +3V3
- U5 pad 6: /USB_D+ -> /USB_D-
Routing:
- net /I2C1_SDA: track 69.4 -> 88.5 mm, vias 6 -> 2
- net /QSPI_SD1: track 18.5 -> 2.14 mm, vias 2 -> 0
- net /QSPI_SD2: track 17.5 -> 2.10 mm, vias 2 -> 0
- net /QSPI_SD0: track 18.5 -> 4.92 mm, vias 2 -> 0
- net /I2C1_SCL: track 70.7 -> 84.2 mm, vias 4 -> 2
- net /TP_DR_Left: track 69.7 -> 82.6 mm, vias 4 -> 2
- net Net-(U2-XIN): track 18.6 -> 6.35 mm, vias 2 -> 0
- net +5V: track 86.1 -> 74.7 mm
- net /QSPI_SD3: track 20.3 -> 9.16 mm, vias 2 -> 0
- net GND: track 52.7 -> 42.3 mm, vias 130 -> 132
- net Net-(J3-CC1): track 72.8 -> 62.8 mm
- net /QSPI_SCLK: track 19.3 -> 10.4 mm, vias 2 -> 0
- net /QSPI_SS: track 24.1 -> 16.1 mm
- net Net-(J3-CC2): track 71.2 -> 63.2 mm
- net /I2C0_SCL: track 292.3 -> 300.3 mm, vias 11 -> 10
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Other:
- board text added: "by rp2040"
