File: flex/quacken.kicad_sch (KiCad schematic)
At the start: 99 parts, among them J1 CIRQUE_Left, J2 CIRQUE_Right, J3 USB_C_Receptacle_USB2.0_16P, U1 W25Q128JVS, U2 RP2040, U3 PCAL6524HEAZ, U4 XC6206PxxxMR, U5 SRV05-4, Y1 12MHz 18pF

Commit message: flex 25.11 (#11)
Parts:
- removed MS1, MS10, MS11, MS12, MS2, MS3, MS4, MS5, MS6, MS7, MS8, MS9: ~, keyboard:MedianPosition, symbol Keyboards:MedianSwitch
- removed R11: 22k, Resistor_SMD:R_0402_1005Metric, symbol Device:R
- added U6: SRV05-4, Package_TO_SOT_SMD:SOT-23-6, symbol Power_Protection:SRV05-4
- R10, R7, R8, R9: value 22k -> 4.7k
- SW1, SW16, SW17, SW2, SW23, SW24, SW25, SW26, SW38, SW39, SW5, SW6: footprint keyboard:PG1350 -> keyboard:Choc_Switch_Median; symbol Keyboards:Switch -> Keyboards:MedianSwitch
- SW10, SW11, SW12, SW13, SW14, SW15, SW18, SW19, SW20, SW21, SW22, SW27, SW28, SW29, SW3, SW30, SW31, SW32, SW33, SW34, SW35, SW36, SW37, SW4, SW40, SW41, SW42, SW7, SW8, SW9: footprint keyboard:PG1350 -> keyboard:Choc_Switch
Connections:
- net +3V3: now also U3.26 (ADDR), U5.5 (VP), U6.5 (VP)
- net +5V: no longer U5.5 (VP)
- net GND: now also U6.2 (VN)
- net I2C0_SCL: now also U6.1 (IO1), U6.4 (IO3)
- net I2C0_SDA: now also U6.3 (IO2), U6.6 (IO4)
Other:
- moved on the sheet: U5

Commit message: flex 25.12
Parts:
- removed U5: SRV05-4, Package_TO_SOT_SMD:SOT-23-6, symbol Power_Protection:SRV05-4
- added C11: 100n, Capacitor_SMD:C_0402_1005Metric_Pad0.74x0.62mm_HandSolder, symbol Device:C_Small
- added C19, C20: 100n, Capacitor_SMD:C_0402_1005Metric, symbol Device:C_Small
- added H1: TentingPuckLeft, keyboard:TentingPuck, symbol Mechanical:MountingHole
- added H10, H11, H12, H3, H4, H5, H6, H7, H8, H9: MountingHole, MountingHole:MountingHole_2.2mm_M2_DIN965_Pad_TopOnly, symbol Mechanical:MountingHole
- added H2: TentingPuckRight, keyboard:TentingPuck, symbol Mechanical:MountingHole
- added J4: Qwiic, Connector_JST:JST_SH_SM04B-SRSS-TB_1x04-1MP_P1.00mm_Horizontal, symbol Connector_Generic:Conn_01x04
- added R11, R2: 2.2k, Resistor_SMD:R_0402_1005Metric, symbol Device:R
- added U5: ECMF02-2AMX6, Package_DFN_QFN:ST_UQFN-6L_1.5x1.7mm_P0.5mm, symbol Power_Protection:ECMF02-2AMX6
- added U7: LTC4311, Package_TO_SOT_SMD:SOT-363_SC-70-6_Handsoldering, symbol Keyboards:LTC4311
- R7, R8: value 4.7k -> 2.2k
- SMDSW1: JLCPCB Part # C455280 -> C720477
- TRRS1, TRRS2: JLCPCB Part # (none) -> C12569
Connections:
- net +3V3: now also TRRS1.R1, TRRS2.R1, C11.1, C19.1, C20.1, J4.3 (Pin_3), R11.1, R2.1, U7.1 (VCC), U7.3 (Enable); no longer TRRS1.R2, TRRS2.R2
- net GND: now also C11.2, C19.2, C20.2, J4.4 (Pin_4), U5.3 (GND), U7.2 (GND), U7.5 (GND)
- net I2C0_SCL: now also U6.6 (IO4), J4.1 (Pin_1), R11.2, U7.6 (BUS1); no longer U6.4 (IO3)
- net I2C0_SDA: now also TRRS1.R2, TRRS2.R2, U6.4 (IO3), J4.2 (Pin_2), R2.2, U7.4 (BUS2); no longer TRRS1.R1, TRRS2.R1, U6.6 (IO4)
- net D+ renamed USB_D+
- net USB_D+: now also U5.6 (D+_out); no longer R3.2
- net D- renamed USB_D-
- net USB_D-: now also U5.5 (D-_out); no longer R4.2
- new net MCU_D+: R3.2, U5.1 (D+_in)
- new net MCU_D-: R4.2, U5.2 (D-_in)
Other:
- moved on the sheet: C15, C17, U6

Commit message: flex 26.01 (#15)
Parts:
- removed C11: 100n, Capacitor_SMD:C_0402_1005Metric_Pad0.74x0.62mm_HandSolder, symbol Device:C_Small
- removed U5: ECMF02-2AMX6, Package_DFN_QFN:ST_UQFN-6L_1.5x1.7mm_P0.5mm, symbol Power_Protection:ECMF02-2AMX6
- removed U7: LTC4311, Package_TO_SOT_SMD:SOT-363_SC-70-6_Handsoldering, symbol Keyboards:LTC4311
- added U5: SRV05-4, Package_TO_SOT_SMD:SOT-23-6, symbol Power_Protection:SRV05-4
- C1, C2: value 27p -> 15p
- SMDSW1: footprint keyboard:small_smd_switch -> Button_Switch_SMD:SW_SPST_TS-1088-xR020
- U1: value W25Q128JVS -> W25Q16JVUX; footprint Package_SO:SOIC-8_5.3x5.3mm_P1.27mm -> Package_SON:Winbond_USON-8-1EP_3x2mm_P0.5mm_EP0.2x1.6mm; symbol Memory_Flash:W25Q128JVS -> Keyboards:W25Q16JVUX; JLCPCB Part # C97521 -> C2843335
- Y1: value 12MHz 18pF -> 12MHz 10pF; MFR.Part # Q22FA23V0041800 -> C20625731
Connections:
- net MCU_D+ is gone; now on net USB_D+: R3.2
- net MCU_D- is gone; now on net USB_D-: R4.2
- net +3V3: now also U5.5 (VP)
- net GND: now also U1.9 (exp), U5.2 (VN)
- net USB_D+: now also U5.3 (IO2), U5.4 (IO3)
- net USB_D-: now also U5.1 (IO1), U5.6 (IO4)
